Commit message: Feat: orchard map & RGBD camera add

File: urdf/ranger_mini.gazebo.xacro (robot description, xacro)
@@ -77,3 +77,31 @@
       <material>Gazebo/Grey</material>
     </gazebo>
+    <!-- ........................... CAMERA PLUGIN ................................... -->
+    <gazebo reference="kinect_camera">
+        <sensor name="kinect_camera" type="depth">
+            <pose> 0 0 0 0 0 0 </pose>
+            <visualize>true</visualize>
+            <update_rate>30</update_rate>
+            <camera>
+                <horizontal_fov>1.089</horizontal_fov>
+                <image>
+                    <format>R8G8B8</format>
+                    <width>640</width>
+                    <height>480</height>
+                </image>
+                <clip>
+                    <near>0.05</near>
+                    <far>8.0</far>
+                </clip>
+            </camera>
+            <plugin name="camera_controller" filename="libgazebo_ros_camera.so">
+                <ros>
+                    <namespace>/</namespace>
+                </ros>
+                <frame_name>kinect_camera_optical</frame_name>
+                <min_depth>0.1</min_depth>
+                <max_depth>100</max_depth>
+            </plugin>
+        </sensor>
+    </gazebo>
 </robot>

File: urdf/ranger_mini.xacro (robot description, xacro)
@@ -474,4 +474,39 @@
       <limit effort="1.5" velocity="20"/>
   </joint>
+  <!-- MACRO -->
+  <xacro:macro name="box_inertia" params="m x y z">
+      <inertia ixx="${m * (y * y + z * z) / 12}" ixy="0" ixz="0" iyy="${m * (x * x + z * z) / 12}" iyz="0" izz="${m * (y * y + x * x) / 12}" />
+  </xacro:macro>
+    <!-- KINECT CAMERA -->
+  <link name="kinect_camera">
+      <collision>
+          <origin xyz="0 0 0" rpy="0 0 0" />
+          <geometry>
+              <box size="0.07 0.3 0.09"/>
+          </geometry>
+      </collision>
+      <visual>
+          <origin xyz="0 0 0" rpy="0 0 0" />
+          <geometry>
+              <mesh filename="file://$(find kimm_orchard_sim)/meshes/kinect/d415.dae"/>
+          </geometry>
+          <material name="black"/>
+      </visual>
+      <inertial>
+          <mass value="0.01"/>
+          <xacro:box_inertia m="0.01" x="0.07" y="0.3" z = "0.09"/>
+      </inertial>
+    </link>
+    <joint name="kinect_camera_joint" type="fixed">
+        <origin rpy="0 0 0" xyz="0.36 0 0.1"/>
+        <parent link="base_link"/>
+        <child link="kinect_camera"/>
+    </joint>
+    <link name="kinect_camera_optical"/>
+    <joint name="kinect_camera_optical_joint" type="fixed">
+        <origin xyz="0 0 0" rpy="${-pi/2} 0 ${-pi/2}"/>
+        <parent link="kinect_camera"/>
+        <child link="kinect_camera_optical"/>
+    </joint>
 	<transmission name="front_left_steering_trans">
       <type>transmission_interface/SimpleTransmission</type>

Commit message: feat: URDF upgrade(IMU, 3D LiDAR add)

File: urdf/ranger_mini.gazebo.xacro (robot description, xacro)
@@ -105,3 +105,24 @@
         </sensor>
     </gazebo>
+    <!-- ........................... IMU PLUGIN ................................... -->
+    <gazebo reference="imu_link">
+      <gravity>true</gravity>
+      <sensor name="imu_sensor" type="imu">
+        <always_on>true</always_on>
+        <update_rate>100</update_rate>
+        <visualize>true</visualize>
+        <topic>__default_topic__</topic>
+        <plugin filename="libgazebo_ros_imu_sensor.so" name="imu_plugin">
+          <topicName>imu</topicName>
+          <bodyName>imu_link</bodyName>
+          <updateRateHZ>10.0</updateRateHZ>
+          <gaussianNoise>0.0</gaussianNoise>
+          <xyzOffset>0 0 0</xyzOffset>
+          <rpyOffset>0 0 0</rpyOffset>
+          <frameName>imu_link</frameName>
+          <initialOrientationAsReference>false</initialOrientationAsReference>
+        </plugin>
+        <pose>0 0 0 0 0 0</pose>
+      </sensor>
+    </gazebo>
 </robot>

File: urdf/ranger_mini.xacro (robot description, xacro)
@@ -662,4 +662,42 @@
     </joint>
   </ros2_control>
+  <!-- IMU -->
+  <link name="imu_link">
+    <collision>
+      <origin xyz="0 0 0" rpy="0 0 0"/>
+      <geometry>
+    <box size="0.00 0.00 0.00"/>
+      </geometry>
+    </collision>
+    <visual>
+      <origin xyz="0 0 0" rpy="0 0 0"/>
+      <geometry>
+    <box size="0.001 0.001 0.001"/>
+      </geometry>
+      <material
+        name="">
+        <color
+          rgba="0.79216 0.81961 0.93333 1" />
+      </material>
+    </visual>
+    <inertial>
+      <mass value="1e-5" />
+      <origin xyz="0 0 0" rpy="0 0 0"/>
+      <inertia ixx="1e-6" ixy="0" ixz="0" iyy="1e-6" iyz="0" izz="1e-6" />
+    </inertial>
+  </link>
+  <joint name="imu_joint" type="fixed">
+    <axis xyz="0 1 0" />
+    <origin xyz="0 0 0" rpy="0 0 0"/>
+    <parent link="base_link"/>
+    <child link="imu_link"/>
+  </joint>
+  <!-- LIDAR -->
+  <xacro:arg name="gpu" default="false"/>
+  <xacro:property name="gpu" value="$(arg gpu)" />
+  <xacro:include filename="$(find kimm_orchard_sim)/urdf/sensors/VLP-16.urdf.xacro"/>
+  <xacro:VLP-16 parent="base_link" name="velodyne" topic="/velodyne_points" hz="10" samples="440" gpu="${gpu}">
+    <origin xyz="0 0 0.18" rpy="0 0 0" />
+  </xacro:VLP-16>
   <gazebo>
     <plugin name="gazebo_ros2_control" filename="libgazebo_ros2_control.so">
