Commit message: feat: ranger mini gazebo control implement

File: urdf/ranger_mini.xacro (robot description, xacro)
@@ -554,6 +554,80 @@
       </actuator>
 	</transmission>
+<ros2_control name="GazeboSystem" type="system">
+    <hardware>
+      <plugin>gazebo_ros2_control/GazeboSystem</plugin>
+    </hardware>
+    <joint name="ffl_wheel_joint">
+      <command_interface name="velocity">
+        <param name="min">-3.14</param>
+        <param name="max">3.14</param>
+      </command_interface>
+      <state_interface name="velocity"/>
+      <state_interface name="effort"/>
+    </joint>
+    <joint name="ffr_wheel_joint">
+      <command_interface name="velocity">
+        <param name="min">-3.14</param>
+        <param name="max">3.14</param>
+      </command_interface>
+      <state_interface name="velocity"/>
+      <state_interface name="effort"/>
+    </joint>
+    <joint name="rfl_wheel_joint">
+      <command_interface name="velocity">
+        <param name="min">-3.14</param>
+        <param name="max">3.14</param>
+      </command_interface>
+      <state_interface name="velocity"/>
+      <state_interface name="effort"/>
+    </joint>
+    <joint name="rfr_wheel_joint">
+      <command_interface name="velocity">
+        <param name="min">-3.14</param>
+        <param name="max">3.14</param>
+      </command_interface>
+      <state_interface name="velocity"/>
+      <state_interface name="effort"/>
+    </joint>
+    <joint name="front_left_steering_joint">
+      <command_interface name="position">
+        <param name="min">-3.14</param>
+        <param name="max">3.14</param>
+      </command_interface>
+      <state_interface name="position"/>
+      <state_interface name="velocity"/>
+      <state_interface name="effort"/>
+    </joint>
+    <joint name="front_right_steering_joint">
+      <command_interface name="position">
+        <param name="min">-3.14</param>
+        <param name="max">3.14</param>
+      </command_interface>
+      <state_interface name="position"/>
+      <state_interface name="velocity"/>
+      <state_interface name="effort"/>
+    </joint>
+    <joint name="rear_left_steering_joint">
+      <command_interface name="position">
+        <param name="min">-3.14</param>
+        <param name="max">3.14</param>
+      </command_interface>
+      <state_interface name="position"/>
+      <state_interface name="velocity"/>
+      <state_interface name="effort"/>
+    </joint>
+    <joint name="rear_right_steering_joint">
+      <command_interface name="position">
+        <param name="min">-3.14</param>
+        <param name="max">3.14</param>
+      </command_interface>
+      <state_interface name="position"/>
+      <state_interface name="velocity"/>
+      <state_interface name="effort"/>
+    </joint>
+  </ros2_control>
   <gazebo>
-    <plugin name="gazebo_ros_control" filename="libgazebo_ros_control.so">
+    <plugin name="gazebo_ros2_control" filename="libgazebo_ros2_control.so">
+      <parameters>/home/minwoo/ros2_ws/install/kimm_orchard_sim/share/kimm_orchard_sim/config/controller.yaml</parameters>
     </plugin>
   </gazebo>

Commit message: ranger_mini -> ranger_mini_v2

File: urdf/ranger_mini.xacro (robot description, xacro)
@@ -1,20 +1,59 @@
 <?xml version="1.0" encoding="utf-8"?>
-<robot name="ranger_mini" xmlns:xacro="http://ros.org/wiki/xacro">
-  <xacro:include filename="$(find kimm_orchard_sim)/urdf/ranger_mini.gazebo.xacro"/>
+<!-- This URDF was automatically created by SolidWorks to URDF Exporter! Originally created by Stephen Brawner (brawner@gmail.com)
+     Commit Version: 1.6.0-4-g7f85cfe  Build Version: 1.6.7995.38578
+     For more information, please see http://wiki.ros.org/sw_urdf_exporter -->
+<robot
+  name="ranger_mini_v2" xmlns:xacro="http://ros.org/wiki/xacro">
+  <xacro:include filename="$(find kimm_orchard_sim)/urdf/ranger_l.xacro" />
+  <xacro:include filename="$(find kimm_orchard_sim)/urdf/ranger_r.xacro" />
+  <!-- Variables -->
+  <xacro:property name="M_PI" value="3.14159"/>
+  <!-- Vehicle Geometries -->
+  <xacro:property name="base_x_size" value="1.0" />
+  <xacro:property name="base_y_size" value="0.380000" />
+  <xacro:property name="base_z_size" value="0.210000" />
+  <xacro:property name="wheelbase" value="0.498" />
+  <xacro:property name="track" value="0.58306" />
+  <xacro:property name="wheel_vertical_offset" value="-0.0702" />
+  <xacro:property name="wheel_length" value="1.1653e-01" />
+  <xacro:property name="wheel_radius" value="1.6459e-01" />
+  <link name="base_link">
+      <inertial>
+          <origin xyz="0.0 0.0 0.0"/>
+          <mass value="10"/>
+          <inertia ixx="1" ixy="0.0" ixz="0.0" iyy="1" iyz="0.0" izz="1"/>
+      </inertial>
+      <visual>
+          <origin xyz="0 0 0" rpy="1.57 0 3.14" />
+          <geometry>
+            <box size="0.5 0.0001 0.2"/>
+          </geometry>
+          <material
+            name="">
+            <color
+            rgba="0.79216 0.81961 0.93333 1" />
+      </material>
+      </visual>
+      <collision>
+          <origin xyz="0 0 -0.1" rpy="0 0 0" />
+          <geometry>
+              <box size="0.5 0.35 0.2"/>
+          </geometry>
+      </collision>
+  </link>
   <link
-    name="base_link">
+    name="ranger_base">
     <inertial>
       <origin
-        xyz="0.0562591525803034 5.21904025701792E-05 0.108402855968814"
-        rpy="0 0 0" />
-      <mass
-        value="17.8446713847014" />
+        xyz="0.00022129 0.05602 -0.18095"
+        rpy="0 0 0" />
       <inertia
-        ixx="0.114563750887795"
-        ixy="1.00505607229726E-06"
-        ixz="-0.00308015585160256"
-        iyy="0.25640701981465"
-        iyz="-1.26769813175445E-06"
-        izz="0.33939943437936" />
+        ixx="1.3986"
+        ixy="0.0052859"
+        ixz="0.00022814"
+        iyy="2.0867"
+        iyz="-0.00025555"
+        izz="0.99513" />
+      <mass value="10"/>
     </inertial>
     <visual>
@@ -24,37 +63,41 @@
       <geometry>
         <mesh
-          filename="file://$(find kimm_orchard_sim)/meshes/base_link.STL" />
+          filename="file://$(find kimm_orchard_sim)/meshes/ranger_mini_v2/base_link.STL" />
       </geometry>
       <material
         name="">
         <color
-          rgba="0.792156862745098 0.819607843137255 0.933333333333333 1" />
+          rgba="0.79216 0.81961 0.93333 1" />
       </material>
     </visual>
-    <collision>
-      <origin
-        xyz="0 0 0"
-        rpy="0 0 0" />
-      <geometry>
-        <mesh
-          filename="file://$(find kimm_orchard_sim)/meshes/base_link.STL" />
-      </geometry>
-    </collision>
   </link>
+  <joint
+    name="base_to_body_joint"
+    type="fixed">
+    <origin
+      xyz="0.2 0.0 -0.1"
+      rpy="0 0 1.57" />
+    <parent
+      link="base_link" />
+    <child
+      link="ranger_base" />
+    <axis
+      xyz="0 0 0" />
+  </joint>
   <link
-    name="front_left_steering_link">
+    name="lidar_connector_link">
     <inertial>
       <origin
-        xyz="-0.0078125 1.2678E-05 0.060941"
+        xyz="-1.6456E-07 0.031388 -0.00014469"
         rpy="0 0 0" />
       <mass
-        value="0.30421" />
+        value="0.29864" />
       <inertia
-        ixx="0.00022406"
-        ixy="-5.3036E-09"
-        ixz="-1.2289E-08"
-        iyy="0.00021285"
-        iyz="-2.5969E-08"
-        izz="0.00027948" />
+        ixx="0.00022074"
+        ixy="-1.5269E-09"
+        ixz="9.9504E-11"
+        iyy="0.00022553"
+        iyz="-9.7446E-07"
+        izz="0.00022125" />
     </inertial>
     <visual>
@@ -64,5 +107,5 @@
       <geometry>
         <mesh
-          filename="file://$(find kimm_orchard_sim)/meshes/front_left_steering_link.STL" />
+          filename="file://$(find kimm_orchard_sim)/meshes/ranger_mini_v2/lidar_link.STL" />
       </geometry>
       <material
@@ -78,37 +121,36 @@
       <geometry>
         <mesh
-          filename="file://$(find kimm_orchard_sim)/meshes/front_left_steering_link.STL" />
+          filename="file://$(find kimm_orchard_sim)/meshes/ranger_mini_v2/lidar_link.STL" />
       </geometry>
     </collision>
   </link>
   <joint
-    name="front_left_steering_joint"
-    type="revolute">
+    name="lidar_joint"
+    type="fixed">
     <origin
-      xyz="0.26366 0.18001 0.0557"
-      rpy="3.1416 0 1.5708" />
+      xyz="-0.003125 0.020748 0.40825"
+      rpy="1.5708 0 0" />
     <parent
-      link="base_link" />
+      link="ranger_base" />
     <child
-      link="front_left_steering_link" />
+      link="lidar_connector_link" />
     <axis
-      xyz="0 0 1" />
-    <limit effort="5" velocity="6.28"  lower="-2.1" upper="2.1" />
+      xyz="0 0 0" />
   </joint>
   <link
-    name="ffl_wheel_link">
+    name="camera_link">
     <inertial>
       <origin
-        xyz="-0.0016559 2.498E-05 -1.1185E-05"
+        xyz="0.0031858 -0.1367 -0.35911"
         rpy="0 0 0" />
       <mass
-        value="1.1363" />
+        value="49.651" />
       <inertia
-        ixx="0.0049366"
-        ixy="-9.2744E-07"
-        ixz="2.0492E-07"
-        iyy="0.002578"
-        iyz="9.052E-08"
-        izz="0.0025791" />
+        ixx="1.9172"
+        ixy="0.0075742"
+        ixz="-0.0001303"
+        iyy="2.3411"
+        iyz="-0.019963"
+        izz="1.3399" />
     </inertial>
     <visual>
@@ -118,5 +160,5 @@
       <geometry>
         <mesh
-          filename="file://$(find kimm_orchard_sim)/meshes/ffl_wheel_link.STL" />
+          filename="file://$(find kimm_orchard_sim)/meshes/ranger_mini_v2/camera_link.STL" />
       </geometry>
       <material
@@ -132,37 +174,36 @@
       <geometry>
         <mesh
-          filename="file://$(find kimm_orchard_sim)/meshes/ffl_wheel_link.STL" />
+          filename="file://$(find kimm_orchard_sim)/meshes/ranger_mini_v2/camera_link.STL" />
       </geometry>
     </collision>
   </link>
   <joint
-    name="ffl_wheel_joint"
-    type="continuous">
+    name="camer_joint"
+    type="fixed">
     <origin
-      xyz="-0.0012329 0.00099823 0.179"
-      rpy="0 0 0" />
+      xyz="-0.0029998 -0.17935 0.19625"
+      rpy="1.5708 0 0" />
     <parent
-      link="front_left_steering_link" />
+      link="ranger_base" />
     <child
-      link="ffl_wheel_link" />
+      link="camera_link" />
     <axis
-      xyz="1 0 0" />
-    <limit effort="1.5" velocity="20"/>
+      xyz="0 0 0" />
   </joint>
   <link
-    name="front_right_steering_link">
+    name="imu_link">
     <inertial>
       <origin
-        xyz="0.0078149 5.813E-06 0.060941"
+        xyz="-0.0032791 -0.0052874 1.901E-06"
         rpy="0 0 0" />
       <mass
-        value="0.30422" />
+        value="0.12486" />
       <inertia
-        ixx="0.00022406"
-        ixy="-6.6817E-09"
-        ixz="7.4999E-08"
-        iyy="0.00021285"
-        iyz="-1.9079E-08"
-        izz="0.00027948" />
+        ixx="6.4634E-05"
+        ixy="-5.4832E-07"
+        ixz="-5.2636E-09"
+        iyy="0.00014266"
+        iyz="-3.4885E-09"
+        izz="8.9183E-05" />
     </inertial>
     <visual>
@@ -172,5 +213,5 @@
       <geometry>
         <mesh
-          filename="file://$(find kimm_orchard_sim)/meshes/front_right_steering_link.STL" />
+          filename="file://$(find kimm_orchard_sim)/meshes/ranger_mini_v2/imu_link.STL" />
       </geometry>
       <material
@@ -186,37 +227,36 @@
       <geometry>
         <mesh
-          filename="file://$(find kimm_orchard_sim)/meshes/front_right_steering_link.STL" />
+          filename="file://$(find kimm_orchard_sim)/meshes/ranger_mini_v2/imu_link.STL" />
       </geometry>
     </collision>
   </link>
   <joint
-    name="front_right_steering_joint"
-    type="revolute">
+    name="imu_joint"
+    type="fixed">
     <origin
-      xyz="0.26366 -0.18 0.0557"
-      rpy="3.1416 0 1.5708" />
+      xyz="-0.003 0.087717 0.25475"
+      rpy="-1.5708 0 -1.5708" />
     <parent
-      link="base_link" />
+      link="ranger_base" />
     <child
-      link="front_right_steering_link" />
+      link="imu_link" />
     <axis
-      xyz="0 0 1" />
-    <limit effort="5" velocity="6.28"  lower="-2.1" upper="2.1" />
+      xyz="0 0 0" />
   </joint>
   <link
-    name="ffr_wheel_link">
+    name="gps_link">
     <inertial>
       <origin
-        xyz="0.0016472 -1.6563E-05 2.7857E-05"
+        xyz="0.0019224 0.0077569 -0.0046042"
         rpy="0 0 0" />
       <mass
-        value="1.1364" />
+        value="0.10935" />
       <inertia
-        ixx="0.0049371"
-        ixy="-9.2722E-07"
-        ixz="-1.9886E-07"
-        iyy="0.0025793"
-        iyz="-6.7378E-08"
-        izz="0.0025805" />
+        ixx="5.0871E-05"
+        ixy="6.5043E-08"
+        ixz="1.6569E-07"
+        iyy="0.0001345"
+        iyz="-1.3697E-08"
+        izz="8.7986E-05" />
     </inertial>
     <visual>
@@ -226,5 +266,5 @@
       <geometry>
         <mesh
-          filename="file://$(find kimm_orchard_sim)/meshes/ffr_wheel_link.STL" />
+          filename="file://$(find kimm_orchard_sim)/meshes/ranger_mini_v2/gps_link.STL" />
       </geometry>
       <material
@@ -240,463 +280,410 @@
       <geometry>
         <mesh
-          filename="file://$(find kimm_orchard_sim)/meshes/ffr_wheel_link.STL" />
+          filename="file://$(find kimm_orchard_sim)/meshes/ranger_mini_v2/gps_link.STL" />
       </geometry>
     </collision>
   </link>
   <joint
-    name="ffr_wheel_joint"
-    type="continuous">
+    name="gps_joint"
+    type="fixed">
     <origin
-      xyz="0.0012238 0 0.179"
-      rpy="0 0 0" />
+      xyz="-0.0010729 0.18638 0.36925"
+      rpy="1.5708 0 -3.1416" />
     <parent
-      link="front_right_steering_link" />
+      link="ranger_base" />
     <child
-      link="ffr_wheel_link" />
+      link="gps_link" />
     <axis
-      xyz="1 0 0" />
-    <limit effort="1.5" velocity="20"/>
+      xyz="0 0 0" />
   </joint>
-  <link
-    name="rear_left_steering_link">
-    <inertial>
-      <origin
-        xyz="-0.0079979 9.6737E-06 0.062261"
-        rpy="0 0 0" />
-      <mass
-        value="0.2968" />
-      <inertia
-        ixx="0.00021788"
-        ixy="-5.0547E-08"
-        ixz="-7.6105E-09"
-        iyy="0.00020665"
-        iyz="1.9139E-08"
-        izz="0.00026712" />
-    </inertial>
-    <visual>
-      <origin
-        xyz="0 0 0"
-        rpy="0 0 0" />
-      <geometry>
-        <mesh
-          filename="file://$(find kimm_orchard_sim)/meshes/rear_left_steering_link.STL" />
-      </geometry>
-      <material
-        name="">
-        <color
-          rgba="0.79216 0.81961 0.93333 1" />
-      </material>
-    </visual>
-    <collision>
-      <origin
-        xyz="0 0 0"
-        rpy="0 0 0" />
-      <geometry>
-        <mesh
-          filename="file://$(find kimm_orchard_sim)/meshes/rear_left_steering_link.STL" />
-      </geometry>
-    </collision>
-  </link>
-  <joint
-    name="rear_left_steering_joint"
-    type="revolute">
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