Commit message: fix : absolute path to relative path, debug

File: map/urdf/orchard_geometry.urdf (robot description, URDF)
Before this commit: robot orchard_world, 1 links, 0 joints
Links:
- link orchard_world_link: geometry collision mesh filename=file:///home/hy/ros2_ws/install/kimm_orchard_sim/share/kimm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; collision mesh filename=file:///home/hy/ros2_ws/install/kimm_orchard_sim/share/kimm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

File: map/urdf/orchard_geometry.urdf.xacro (robot description, xacro)
@@ -1,5 +1,4 @@
 <?xml version="1.0"?>
 <robot name="orchard_world" xmlns:xacro="http://www.ros.org/wiki/xacro">
-  <xacro:include filename="$(find kimm_orchard_sim)/urdf/gazebo.xacro"/>
   <link name="orchard_world_link">
     <inertial>

File: urdf/ranger_mini.xacro (robot description, xacro)
@@ -702,5 +702,5 @@
   <gazebo>
     <plugin name="gazebo_ros2_control" filename="libgazebo_ros2_control.so">
-      <parameters>/home/minwoo/ros2_ws/install/kimm_orchard_sim/share/kimm_orchard_sim/config/controller.yaml</parameters>
+      <parameters>$(find kimm_orchard_sim)/config/controller.yaml</parameters>
     </plugin>
   </gazebo>

Commit message: feat: sensors add, config file made

File: map/urdf/orchard_geometry.urdf (robot description, URDF)
Before this commit: robot orchard_world, 1 links, 0 joints
Links:
- link orchard_world_link: geometry collision mesh filename=file:///root/ros2_ws/install/kimm_orchard_sim/share/kimm_or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; collision mesh filename=file:///root/ros2_ws/install/kimm_orchard_sim/share/kimm_or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

File: urdf/ranger_mini.gazebo.xacro (robot description, xacro)
@@ -77,52 +77,2 @@
       <material>Gazebo/Grey</material>
     </gazebo>
-    <!-- ........................... CAMERA PLUGIN ................................... -->
-    <gazebo reference="kinect_camera">
-        <sensor name="kinect_camera" type="depth">
-            <pose> 0 0 0 0 0 0 </pose>
-            <visualize>true</visualize>
-            <update_rate>30</update_rate>
-            <camera>
-                <horizontal_fov>1.089</horizontal_fov>
-                <image>
-                    <format>R8G8B8</format>
-                    <width>640</width>
-                    <height>480</height>
-                </image>
-                <clip>
-                    <near>0.05</near>
-                    <far>8.0</far>
-                </clip>
-            </camera>
-            <plugin name="camera_controller" filename="libgazebo_ros_camera.so">
-                <ros>
-                    <namespace>/</namespace>
-                </ros>
-                <frame_name>kinect_camera_optical</frame_name>
-                <min_depth>0.1</min_depth>
-                <max_depth>100</max_depth>
-            </plugin>
-        </sensor>
-    </gazebo>
-    <!-- ........................... IMU PLUGIN ................................... -->
-    <gazebo reference="imu_link">
-      <gravity>true</gravity>
-      <sensor name="imu_sensor" type="imu">
-        <always_on>true</always_on>
-        <update_rate>300</update_rate>
-        <visualize>true</visualize>
-        <topic>__default_topic__</topic>
-        <plugin filename="libgazebo_ros_imu_sensor.so" name="imu_plugin">
-          <topicName>imu</topicName>
-          <bodyName>imu_link</bodyName>
-          <updateRateHZ>300.0</updateRateHZ>
-          <gaussianNoise>0.0</gaussianNoise>
-          <xyzOffset>0 0 0</xyzOffset>
-          <rpyOffset>0 0 0</rpyOffset>
-          <frameName>imu_link</frameName>
-          <initialOrientationAsReference>false</initialOrientationAsReference>
-        </plugin>
-        <pose>0 0 0 0 0 0</pose>
-      </sensor>
-    </gazebo>
-</robot>

File: urdf/ranger_mini.xacro (robot description, xacro)
@@ -25,5 +25,5 @@
       </inertial>
       <visual>
-          <origin xyz="0 0 0" rpy="1.57 0 3.14" />
+          <origin xyz="0 0 0" rpy="0 0 0" />
           <geometry>
             <box size="0.5 0.0001 0.2"/>
@@ -32,5 +32,5 @@
             name="">
             <color
-            rgba="0.79216 0.81961 0.93333 1" />
+            rgba="0.784 0.784 0.784 1" />
       </material>
       </visual>
@@ -68,5 +68,5 @@
         name="">
         <color
-          rgba="0.79216 0.81961 0.93333 1" />
+          rgba="0.784 0.784 0.784 1" />
       </material>
     </visual>
@@ -112,5 +112,5 @@
         name="">
         <color
-          rgba="0.79216 0.81961 0.93333 1" />
+          rgba="0.314 0.314 0.314 1" />
       </material>
     </visual>
@@ -165,5 +165,5 @@
         name="">
         <color
-          rgba="0.79216 0.81961 0.93333 1" />
+          rgba="0.314 0.314 0.314 1" />
       </material>
     </visual>
@@ -218,5 +218,5 @@
         name="">
         <color
-          rgba="0.79216 0.81961 0.93333 1" />
+          rgba="0.784 0.784 0.784 1" />
       </material>
     </visual>
@@ -271,5 +271,5 @@
         name="">
         <color
-          rgba="0.79216 0.81961 0.93333 1" />
+          rgba="0.9 0.9 0.9 1" />
       </material>
     </visual>
@@ -680,11 +680,19 @@
       </joint>
   </ros2_control>
+  <!-- MACRO -->
+  <xacro:macro name="box_inertia" params="m x y z">
+      <inertia ixx="${m * (y * y + z * z) / 12}" ixy="0" ixz="0" iyy="${m * (x * x + z * z) / 12}" iyz="0" izz="${m * (y * y + x * x) / 12}" />
+  </xacro:macro>
   <!-- LIDAR -->
-  <xacro:arg name="gpu" default="false"/>
-  <xacro:property name="gpu" value="$(arg gpu)" />
-  <xacro:include filename="$(find kimm_orchard_sim)/urdf/sensors/VLP-16.urdf.xacro"/>
-  <xacro:VLP-16 parent="lidar_connector_link" name="velodyne" topic="/velodyne_points" hz="10" samples="440" gpu="${gpu}">
+  <xacro:include filename="$(find kimm_orchard_sim)/urdf/sensors/VLP-32.urdf.xacro"/>
+  <xacro:VLP-32 >
     <origin xyz="0 0 0" rpy="-1.57 -1.57 0.0" />
-  </xacro:VLP-16>
+  </xacro:VLP-32>
+  <!-- CAMERA -->
+  <xacro:include filename="$(find kimm_orchard_sim)/urdf/sensors/kinect_camera.xacro" />
+  <xacro:kinect_camera />
+  <!-- IMY -->
+  <xacro:include filename="$(find kimm_orchard_sim)/urdf/sensors/imu.xacro" />
+  <xacro:imu />
   <gazebo>
     <plugin name="gazebo_ros2_control" filename="libgazebo_ros2_control.so">

File: urdf/sensors/VLP-32.urdf.xacro (robot description, xacro)
@@ -1,6 +1,23 @@
 <?xml version="1.0"?>
-<robot xmlns:xacro="http://www.ros.org/wiki/xacro" name="VLP-16">
+<robot xmlns:xacro="http://www.ros.org/wiki/xacro" name="VLP-32">
   <xacro:property name="M_PI" value="3.1415926535897931" />
-  <xacro:macro name="VLP-16" params="*origin parent:=base_link name:=velodyne topic:=/velodyne_points hz:=10 lasers:=16 samples:=1875 collision_range:=0.3 min_range:=0.9 max_range:=130.0 noise:=0.008 min_angle:=-${M_PI} max_angle:=${M_PI} gpu:=false">
+  <xacro:macro name="VLP-32" params="*origin">
+  <xacro:property name="yaml_path" value="$(find kimm_orchard_sim)/config/sensor_params.yaml" />
+  <xacro:property name="dict_yaml" value="${xacro.load_yaml(yaml_path)}" />
+  <!-- lidar parameters -->
+  <xacro:property name="lidar" value="${dict_yaml['lidar']}" />
+  <xacro:property name="parent" value="${lidar['parent']}" />
+  <xacro:property name="name" value="${lidar['name']}" />
+  <xacro:property name="topic" value="${lidar['topic']}" />
+  <xacro:property name="hz" value="${lidar['hz']}" />
+  <xacro:property name="lasers" value="${lidar['lasers']}" />
+  <xacro:property name="samples" value="${lidar['samples']}" />
+  <xacro:property name="collision_range" value="${lidar['collision_range']}" />
+  <xacro:property name="min_range" value="${lidar['min_range']}" />
+  <xacro:property name="max_range" value="${lidar['max_range']}" />
+  <xacro:property name="noise" value="${lidar['noise']}" />
+  <xacro:property name="min_angle" value="${lidar['min_angle']}" />
+  <xacro:property name="max_angle" value="${lidar['max_angle']}" />
+  <xacro:property name="gpu" value="${lidar['gpu']}" />
     <joint name="${name}_base_mount_joint" type="fixed">
       <xacro:insert_block name="origin" />
@@ -9,27 +26,4 @@
     </joint>
     <link name="${name}_base_link">
-      <inertial>
-        <mass value="0.83"/>
-        <origin xyz="0 0 0.03585"/>
-        <inertia ixx="${(0.83 * (3.0*0.0516*0.0516 + 0.0717*0.0717)) / 12.0}" ixy="0" ixz="0"
-          iyy="${(0.83 * (3.0*0.0516*0.0516 + 0.0717*0.0717)) / 12.0}" iyz="0"
-          izz="${0.5 * 0.83 * (0.0516*0.0516)}"/>
-      </inertial>
-      <visual>
-        <geometry>
-          <mesh filename="$(find kimm_orchard_sim)/meshes/lidar/VLP16_base_1.dae" />
-        </geometry>
-      </visual>
-      <visual>
-        <geometry>
-          <mesh filename="$(find kimm_orchard_sim)/meshes/lidar/VLP16_base_2.dae" />
-        </geometry>
-      </visual>
-      <collision>
-        <origin rpy="0 0 0" xyz="0 0 0.03585"/>
-        <geometry>
-          <cylinder radius="0.0516" length="0.0717"/>
-        </geometry>
-      </collision>
     </link>
     <joint name="${name}_base_scan_joint" type="fixed" >
@@ -39,15 +33,4 @@
     </joint>
     <link name="${name}">
-      <inertial>
-        <mass value="0.01"/>
-        <origin xyz="0 0 0"/>
-        <inertia ixx="1e-7" ixy="0" ixz="0" iyy="1e-7" iyz="0" izz="1e-7"/>
-      </inertial>
-      <visual>
-        <origin xyz="0 0 -0.0377" />
-        <geometry>
-          <mesh filename="$(find kimm_orchard_sim)/meshes/lidar/VLP16_scan.dae" />
-        </geometry>
-      </visual>
     </link>
     <!-- Gazebo requires the velodyne_gazebo_plugins package -->
