Commit message: feat:robot_localization

File: LIO-SAM/config/robot.urdf.xacro (robot description, xacro)
@@ -9,20 +9,38 @@
     <origin xyz="0 0 0" rpy="0 0 0" />
   </joint>
-  <link name="lidar_link"> </link>
+  <link name="laser_data_frame"> </link>
   <joint name="lidar_joint" type="fixed">
     <parent link="base_link" />
-    <child link="lidar_link" />
+    <child link="laser_data_frame" />
+    <origin xyz="0 0 0" rpy="0 0 3.141592" />
+  </joint>
+  <link name="imu_data_frame"> </link>
+  <joint name="lidar_imu_joint" type="fixed">
+    <parent link="laser_data_frame" />
+    <child link="imu_data_frame" />
     <origin xyz="0 0 0" rpy="0 0 0" />
   </joint>
-  <link name="imu_link"> </link>
-  <joint name="imu_joint" type="fixed">
-    <parent link="chassis_link" />
-    <child link="imu_link" />
+  <link name="imu_seu"> </link>
+  <joint name="imu_seu_joint" type="fixed">
+    <parent link="base_link" />
+    <child link="imu_seu" />
     <origin xyz="0 0 0" rpy="0 0 0" />
   </joint>
-  <link name="laser_sensor_frame"> </link>
-  <joint name="laser_joint" type="fixed">
-    <parent link="imu_link" />
-    <child link="laser_sensor_frame" />
+  <link name="imu_enu"> </link>
+  <joint name="imu_enu_joint" type="fixed">
+    <parent link="base_link" />
+    <child link="imu_enu" />
+    <origin xyz="0 0 0" rpy="0 0 0"/> <!-- 3.141592 3.141592 1.5708" /> -->
+  </joint>
+  <link name="imu_ned"> </link>
+  <joint name="imu_ned_joint" type="fixed">
+    <parent link="base_link" />
+    <child link="imu_ned" />
+    <origin xyz="0 0 0" rpy="0 3.141592 0" />
+  </joint>
+  <link name="gps"> </link>
+  <joint name="gps_joint" type="fixed">
+    <parent link="base_link" />
+    <child link="gps" />
     <origin xyz="0 0 0" rpy="0 0 0" />
   </joint>

File: kimm_orchard_sim/urdf/sensors/VLP-32.urdf.xacro (robot description, xacro)
@@ -29,5 +29,5 @@
     </link>
     <joint name="${name}_base_scan_joint" type="fixed" >
-      <origin xyz="0 0 0.0377" rpy="0 0 0" />
+      <origin xyz="0 0 -0.4" rpy="0 0 0" />
       <parent link="${name}_base_link" />
       <child link="${name}"/>

Commit message: edit slam code

File: LIO-SAM/config/robot.urdf.xacro (robot description, xacro)
@@ -9,38 +9,20 @@
     <origin xyz="0 0 0" rpy="0 0 0" />
   </joint>
-  <link name="laser_data_frame"> </link>
+  <link name="lidar_link"> </link>
   <joint name="lidar_joint" type="fixed">
     <parent link="base_link" />
-    <child link="laser_data_frame" />
-    <origin xyz="0 0 0" rpy="0 0 3.141592" />
-  </joint>
-  <link name="imu_data_frame"> </link>
-  <joint name="lidar_imu_joint" type="fixed">
-    <parent link="laser_data_frame" />
-    <child link="imu_data_frame" />
+    <child link="lidar_link" />
     <origin xyz="0 0 0" rpy="0 0 0" />
   </joint>
-  <link name="imu_seu"> </link>
-  <joint name="imu_seu_joint" type="fixed">
-    <parent link="base_link" />
-    <child link="imu_seu" />
+  <link name="imu_link"> </link>
+  <joint name="imu_joint" type="fixed">
+    <parent link="chassis_link" />
+    <child link="imu_link" />
     <origin xyz="0 0 0" rpy="0 0 0" />
   </joint>
-  <link name="imu_enu"> </link>
-  <joint name="imu_enu_joint" type="fixed">
-    <parent link="base_link" />
-    <child link="imu_enu" />
-    <origin xyz="0 0 0" rpy="0 0 0"/> <!-- 3.141592 3.141592 1.5708" /> -->
-  </joint>
-  <link name="imu_ned"> </link>
-  <joint name="imu_ned_joint" type="fixed">
-    <parent link="base_link" />
-    <child link="imu_ned" />
-    <origin xyz="0 0 0" rpy="0 3.141592 0" />
-  </joint>
-  <link name="gps"> </link>
-  <joint name="gps_joint" type="fixed">
-    <parent link="base_link" />
-    <child link="gps" />
+  <link name="laser_sensor_frame"> </link>
+  <joint name="laser_joint" type="fixed">
+    <parent link="imu_link" />
+    <child link="laser_sensor_frame" />
     <origin xyz="0 0 0" rpy="0 0 0" />
   </joint>
